Commit message: arm spawning in gazebo

File: src/scoutbot_description/urdf/arm.urdf.xacro (robot description, xacro)
@@ -8,4 +8,5 @@
   <!--Base Link-->
   <gazebo>
+    <static> true </static>
     <plugin name="gazebo_ros2_control" filename="libgazebo_ros2_control.so"/>
   </gazebo>
@@ -39,5 +40,5 @@
       <origin xyz="0 0 0" rpy="${1.5708} 0 0"/>
       <geometry>
-        <mesh filename="package://scoutbot_description/meshes/Base.stl" scale="${mesh_scale}"/>
+        <mesh filename="/home/bbhanda/scoutbot_ws/src/scoutbot_description/meshes/Base.stl" scale="${mesh_scale}"/>
       </geometry>
       <material name="grey"/>
@@ -48,5 +49,5 @@
       <origin xyz="0 0 0" rpy="${1.5708} 0 0"/>
       <geometry>
-        <mesh filename="package://scoutbot_description/meshes/Base_Cover.stl" scale="${mesh_scale}"/>
+        <mesh filename="/home/bbhanda/scoutbot_ws/src/scoutbot_description/meshes/Base_Cover.stl" scale="${mesh_scale}"/>
       </geometry>
       <material name="grey"/>
@@ -76,5 +77,5 @@
       <origin xyz="0 0 0" rpy="${-1.5708} 0 0"/>
       <geometry>
-        <mesh filename="package://scoutbot_description/meshes/Joint_1.stl" scale="${mesh_scale}"/>
+        <mesh filename="/home/bbhanda/scoutbot_ws/src/scoutbot_description/meshes/Joint_1.stl" scale="${mesh_scale}"/>
       </geometry>
       <material name="grey"/>
@@ -104,5 +105,5 @@
       <origin xyz="0 0 0" rpy="${1.5708} 0 0"/>
       <geometry>
-        <mesh filename="package://scoutbot_description/meshes/Link_1-Joint_2.stl" scale="${mesh_scale}"/>
+        <mesh filename="/home/bbhanda/scoutbot_ws/src/scoutbot_description/meshes/Link_1-Joint_2.stl" scale="${mesh_scale}"/>
       </geometry>
       <material name="grey"/>
@@ -148,5 +149,5 @@
       <origin xyz="-0.5 0 0" rpy="0 1.5708 0"/>
       <geometry>
-        <mesh filename="package://scoutbot_description/meshes/Link_2-Joint_3.stl" scale="${mesh_scale}"/>
+        <mesh filename="/home/bbhanda/scoutbot_ws/src/scoutbot_description/meshes/Link_2-Joint_3.stl" scale="${mesh_scale}"/>
       </geometry>
       <material name="grey"/>
@@ -192,5 +193,5 @@
       <origin xyz="-0.70 -0.20 0.1" rpy="0 1.7508 0"/>
       <geometry>
-        <mesh filename="package://scoutbot_description/meshes/Link_3-Joint_4.stl" scale="${mesh_scale}"/>
+        <mesh filename="/home/bbhanda/scoutbot_ws/src/scoutbot_description/meshes/Link_3-Joint_4.stl" scale="${mesh_scale}"/>
       </geometry>
       <material name="grey"/>
@@ -236,5 +237,5 @@
       <origin xyz="-0.4 0 0" rpy="0.2 0 1.5708"/>
       <geometry>
-        <mesh filename="package://scoutbot_description/meshes/Link_4-Joint_5.stl" scale="${mesh_scale}"/>
+        <mesh filename="/home/bbhanda/scoutbot_ws/src/scoutbot_description/meshes/Link_4-Joint_5.stl" scale="${mesh_scale}"/>
       </geometry>
       <material name="grey"/>
@@ -278,7 +279,7 @@
   <link name="Joint_6">
     <visual>
-      <origin xyz="0 0 0" rpy="0 0 0"/>
-      <geometry>
-        <mesh filename="package://scoutbot_description/meshes/Link_5-Joint_6.stl" scale="${mesh_scale}"/>
+      <origin xyz="-0.4 0 0" rpy="0.005 0 -1.5708"/>
+      <geometry>
+        <mesh filename="/home/bbhanda/scoutbot_ws/src/scoutbot_description/meshes/Link_5-Joint_6.stl" scale="${mesh_scale}"/>
       </geometry>
       <material name="grey"/>
